Commit message: load sawback urdf into robot_description

File: urdf/nwu03_ridgeback_extras.urdf.xacro (robot description, xacro)
@@ -28,5 +28,5 @@
      <visual>
       <geometry>
-        <mesh filename="package://nwu03_ridgeback/meshes/vlp16_assy.stl"/>
+        <mesh filename="package://nu_ridgeback/meshes/vlp16_assy.stl"/>
       </geometry>
       <material name="light_grey">
@@ -36,5 +36,5 @@
     <collision>
       <geometry>
-        <mesh filename="package://nwu03_ridgeback/meshes/vlp16_assy.stl"/>
+        <mesh filename="package://nu_ridgeback/meshes/vlp16_assy.stl"/>
       </geometry>
     </collision>
@@ -56,5 +56,5 @@
      <visual>
       <geometry>
-        <mesh filename="package://nwu03_ridgeback/meshes/bb2_stereo_cam.dae"/>
+        <mesh filename="package://nu_ridgeback/meshes/bb2_stereo_cam.dae"/>
       </geometry>
     </visual>
