Commit message: move base forward in urdf

File: nuridgeback_description/urdf/sawyer_mount.urdf.xacro (robot description, xacro)
@@ -25,5 +25,5 @@
   </link>
   <joint name="mount_joint" type="fixed">
-    <origin rpy="0 0 0" xyz="0.19 0.0 0.280"/>
+    <origin rpy="0 0 0" xyz="0.205 0.0 0.280"/>
     <parent link="base_link"/>
     <child link="mount_link"/>
