Commit message: rtabmap_ros setup and config

File: nuridgeback_description/urdf/bumblebee_camera.urdf.xacro (robot description, xacro)
@@ -21,4 +21,5 @@
    <origin xyz="0.001 0 0.07" rpy="0 0 ${-1.5708}" />
  </joint>
+ <!-- <link name="bb2_optical_link" /> -->
  <link name="bb2_optical_link" />
  <joint name="bb2_origin_to_bb2_camera" type="fixed">

Commit message: add link for left optical frame

File: nuridgeback_description/urdf/bumblebee_camera.urdf.xacro (robot description, xacro)
@@ -12,5 +12,5 @@
    <parent link="mid_mount" />
    <child link="bb2_mesh" />
-   <origin xyz="0.43 0 0" rpy="0 0 1.5708" />
+   <origin xyz="0.43 0 0" rpy="0.663 0 1.5708" />
  </joint>
  <!-- Create a link between the BB2 mesh and sensor origin -->
@@ -21,10 +21,15 @@
    <origin xyz="0.001 0 0.07" rpy="0 0 ${-1.5708}" />
  </joint>
- <!-- <link name="bb2_optical_link" /> -->
  <link name="bb2_optical_link" />
  <joint name="bb2_origin_to_bb2_camera" type="fixed">
    <parent link="bb2_origin" />
    <child link="bb2_optical_link" />
-   <origin xyz="0.01 0 0" rpy="${-1.5708} 0 ${-1.5708}" />
+   <origin xyz="0 0 0" rpy="${-1.5708} 0 ${-1.5708}" />
+ </joint>
+ <link name="bb2_left_optical_link" />
+ <joint name="bb2_left_optical_joint" type="fixed">
+   <parent link="bb2_optical_link" />
+   <child link="bb2_left_optical_link" />
+   <origin xyz="-0.06 0 0" rpy="0 0 0" />
  </joint>
 </robot>

Commit message: added gazebo plugin for sensor simulation

File: nuridgeback_description/urdf/bumblebee_camera.urdf.xacro (robot description, xacro)
@@ -1,4 +1,48 @@
 <?xml version="1.0"?>
 <robot xmlns:xacro="http://ros.org/wiki/xacro">
+  <xacro:macro name="BB2" params="camera_link:=bb2_origin camera_optical_link:=bb2_optical_link">
+     <gazebo reference="${camera_link}">
+       <sensor name="bumblebee" type="depth">
+         <update_rate>30</update_rate>
+         <camera>
+           <pose>0 0 0 0 0 0</pose>
+           <horizontal_fov>1.047198</horizontal_fov>
+           <image>
+             <width>640</width>
+             <height>480</height>
+             <format>R8G8B8</format>
+           </image>
+           <clip>
+             <near>0.05</near>
+             <far>3</far>
+           </clip>
+         </camera>
+         <plugin name="bumblebee_controller" filename="libgazebo_ros_openni_kinect.so">
+           <baseline>0.2</baseline>
+           <alwaysOn>true</alwaysOn>
+           <updateRate>1.0</updateRate>
+           <cameraName>bumblebee</cameraName>
+           <imageTopicName>color/image_raw</imageTopicName>
+           <cameraInfoTopicName>color/camera_info</cameraInfoTopicName>
+           <depthImageTopicName>depth/image_raw</depthImageTopicName>
+           <depthImageInfoTopicName>depth/camera_info</depthImageInfoTopicName>
+           <pointCloudTopicName>depth/points</pointCloudTopicName>
+           <frameName>${camera_optical_link}</frameName>
+           <pointCloudCutoff>0.5</pointCloudCutoff>
+           <pointCloudCutoffMax>3.0</pointCloudCutoffMax>
+           <distortionK1>0.00000001</distortionK1>
+           <distortionK2>0.00000001</distortionK2>
+           <distortionK3>0.00000001</distortionK3>
+           <distortionT1>0.00000001</distortionT1>
+           <distortionT2>0.00000001</distortionT2>
+           <CxPrime>0</CxPrime>
+           <Cx>0</Cx>
+           <Cy>0</Cy>
+           <focalLength>0</focalLength>
+           <hackBaseline>0</hackBaseline>
+         </plugin>
+       </sensor>
+     </gazebo>
+   </xacro:macro>
 <!-- Create link for Bumblebee mesh -->
  <link name="bb2_mesh">
@@ -33,3 +77,4 @@
    <origin xyz="-0.06 0 0" rpy="0 0 0" />
  </joint>
+ <xacro:BB2 camera_link="bb2_origin" camera_optical_link="bb2_optical_link"/>
 </robot>

File: nuridgeback_description/urdf/velodyne.urdf.xacro (robot description, xacro)
@@ -1,4 +1,48 @@
 <?xml version="1.0"?>
 <robot xmlns:xacro="http://ros.org/wiki/xacro">
+  <xacro:property name="M_PI" value="3.1415926535897931" />
+  <xacro:macro name="VLP-16" params="name:=velodyne topic:=velodyne_points">
+    <!-- Gazebo requires the velodyne_gazebo_plugins package -->
+    <gazebo reference="${name}">
+      <sensor type="ray" name="${name}-VLP16">
+        <pose>0 0 0 0 0 0</pose>
+        <visualize>false</visualize>
+        <update_rate>10</update_rate>
+        <ray>
+          <scan>
+            <horizontal>
+              <samples>1875</samples>
+              <resolution>1</resolution>
+              <min_angle>${-1.0*M_PI}</min_angle>
+              <max_angle>${M_PI}</max_angle>
+            </horizontal>
+            <vertical>
+              <samples>16</samples>
+              <resolution>1</resolution>
+              <min_angle>-${15.0*M_PI/180.0}</min_angle>
+              <max_angle> ${15.0*M_PI/180.0}</max_angle>
+            </vertical>
+          </scan>
+          <range>
+            <min>0.3</min>
+            <max>${130.0+1.0}</max>
+            <resolution>0.001</resolution>
+          </range>
+          <noise>
+            <type>gaussian</type>
+            <mean>0.0</mean>
+            <stddev>0.0</stddev>
+          </noise>
+        </ray>
+        <plugin name="gazebo_ros_laser_controller" filename="libgazebo_ros_velodyne_laser.so">
+          <topicName>${topic}</topicName>
+      	  <frameName>${name}</frameName>
+          <min_range>0.9</min_range>
+          <max_range>130.0</max_range>
+          <gaussianNoise>0.008</gaussianNoise>
+        </plugin>
+      </sensor>
+    </gazebo>
+  </xacro:macro>
   <!-- Create link for VLP16 mesh  -->
   <link name="velodyne_mesh">
@@ -29,3 +73,4 @@
     <origin xyz="0 0 0.195" rpy="0 0 0" />
   </joint>
+  <xacro:VLP-16 name="velodyne_scan" topic="velodyne_points"/>
 </robot>
